File: camCAD/camCAD.kicad_sch (KiCad schematic)
At the start: 8 parts, among them J1 ILI9341_Display_Header, U1 STM32F407ZGTx(6)

Commit message: Debug + MicroSD connections complete
Parts:
- added J2: SWD Header, symbol Connector:Conn_01x02_Pin
- U1: value STM32F407ZGTx(6) -> STM32F407ZGT6 LQFP144
Connections:
- net GND: now also U1.107 (VSS), U1.120 (VSS), U1.130 (VSS), U1.16 (VSS), U1.31 (VSSA), U1.38 (VSS), U1.51 (VSS), U1.61 (VSS), U1.83 (VSS), U1.94 (VSS)
- net at OV1.P$1 (RESET): now also U1.58 (PE7)
- net at OV1.P$18 (PWDWN): now also U1.59 (PE8)
- net at Z1.1 (CD): now also U1.46 (PB0)
- net at D1.2 (A): now also U1.114 (PD0)
- net at U1.105 (PA13): now also J2.1 (Pin_1)
- net at U1.109 (PA14): now also J2.2 (Pin_2)
- net at U1.144 (VDD): now also U1.33 (VDDA)
- no-connect marks 123 -> 115
Other:
- note added: "*TODO* 1. ADD POWER SUPPLY (3.3V-3.6V)"
- note added: "CD - GPIO PB0"
- note added: "GPIO PD0"
- note added: "RST - PE7 PWDWN - PE8"
- note added: "SWCLK"
- note added: "SWDIO"
- note removed: "*TODO* 1. ASSIGN GPIO PINS 2. ADD POWER SUPPLY (most likely 3.3V) 3. Add way to flash binaries"
- note removed: "Hook up CD(card detect) to GPIO input"
- note removed: "Hook up RST and PWDWN to GPIO output"
- note removed: "Hook up to GPIO output"
- moved on the sheet: D1, D2, OV1, R1, R2, Z1

Commit message: Finished connections for ILI9341, power incomplete
Connections:
- net at J2.1 (Pin_1): now also U1.111 (PC10); no longer U1.105 (PA13)
- net at J2.2 (Pin_2): now also U1.112 (PC11); no longer U1.109 (PA14)
- net at U1.100 (PA8): now also J1.10
- net at U1.101 (PA9): now also J1.11
- net at U1.133 (PB3): now also J1.9
- net at U1.135 (PB5): now also J1.6
- net at U1.36 (PA2): now also J1.5
- net at U1.37 (PA3): now also J1.4
- no-connect marks 115 -> 108
Other:
- note added: "*TODO* 1. ADD POWER SUPPLY (3.3V-3.6V) 2. More indicator LEDs? 3. Flash?"
- note added: "Actual Product: 1987-DT024ETFT-IPS-SHB-ND 3-Line 9-bit Serial Comms IM[1:0] = 01; IM1(PA9) = LOW, IM0(PA8) = HIGH Using SPI3, RESET bound to PA2 GPIO"
- note removed: "*TODO* 1. ADD POWER SUPPLY (3.3V-3.6V)"
- note removed: "3-Line 9-bit Serial Comms IM[1:0] = 01"
- moved on the sheet: D2, J1, J2, R2

Commit message: Push before adding power configuration
Parts:
- removed D2: PowerLED, symbol Device:LED
- removed R2: 6.8K, symbol Device:R_Small_US
- added C14, C15: 2.2uF, symbol Device:C_Small
- added D3: OVLED, symbol Device:LED
- added D4: SDLED, symbol Device:LED
- added LED1: Activity+PowerLED, CLMVC-FKA-CL1D1L71BB7C3C3_CRE, symbol CLMVC_FKA_CL1D1L71BB7C3C3:CLMVC-FKA-CL1D1L71BB7C3C3
- added R3, R4, R5, R6, R7: 6.8K, symbol Device:R_Small_US
- D1: value ActivityLED -> ExtraLED
Connections:
- net +3.3V: now also LED1.1 (A)
- net GND: now also D1.1 (K), C14.1, C15.1, D3.1 (K), D4.1 (K); no longer R1.2, U1.107 (VSS), U1.120 (VSS), U1.130 (VSS), U1.16 (VSS), U1.31 (VSSA), U1.38 (VSS), U1.51 (VSS), U1.61 (VSS), U1.83 (VSS), U1.94 (VSS)
- net at R1.1: now also U1.114 (PD0); no longer D1.1 (K)
- net at D1.2 (A): now also R1.2; no longer U1.114 (PD0)
- net at U1.106 (VCAP_2): now also C15.2
- net at U1.115 (PD1): now also R3.1
- net at U1.116 (PD2): now also R4.1
- net at U1.144 (VDD): no longer U1.33 (VDDA)
- net at U1.71 (VCAP_1): now also C14.2
- net at U1.81 (PD12): now also R5.1
- net at U1.82 (PD13): now also R6.1
- net at U1.85 (PD14): now also R7.1
- new net: D3.2 (A), R3.2
- new net: U1.107 (VSS), U1.120 (VSS), U1.130 (VSS), U1.16 (VSS), U1.38 (VSS), U1.51 (VSS), U1.61 (VSS), U1.83 (VSS), U1.94 (VSS)
- new net: LED1.3 (G), R6.2
- new net: D4.2 (A), R4.2
- new net: LED1.2 (B), R5.2
- new net: LED1.4 (R), R7.2
- no-connect marks 108 -> 89
Other:
- note added: "TODO: 1. Add power supply 2. Assign XCLK 3. Calculate RGB LED Resistor values"
- note removed: "*TODO* 1. ADD POWER SUPPLY (3.3V-3.6V) 2. More indicator LEDs? 3. Flash?"
- note removed: "GPIO PD0"
- moved on the sheet: D1, OV1, R1

Commit message: working on power
Parts:
- removed C14, C15: 2.2uF, symbol Device:C_Small
- removed D1: ExtraLED, symbol Device:LED
- removed D3: OVLED, symbol Device:LED
- removed D4: SDLED, symbol Device:LED
- removed J1: ILI9341_Display_Header, 5051101592:CON_5051101592_MOL, symbol 1_Headers:5051101592
- removed J2: SWD Header, symbol Connector:Conn_01x02_Pin
- removed LED1: Activity+PowerLED, CLMVC-FKA-CL1D1L71BB7C3C3_CRE, symbol CLMVC_FKA_CL1D1L71BB7C3C3:CLMVC-FKA-CL1D1L71BB7C3C3
- removed OV1: CAMERA-OV7670, CAMERA-OV7670:CAMERA-OV7670-DIP, symbol 1_Cameras:CAMERA-OV7670
- removed R1, R3, R4, R5, R6, R7: 6.8K, symbol Device:R_Small_US
- removed U1: STM32F407ZGT6 LQFP144, Package_QFP:LQFP-144_20x20mm_P0.5mm, symbol MCU_ST_STM32F4:STM32F407ZGTx
- removed Z1: MicroSD_Breakout, symbol 1_MicroSD:MicroSD_BREA
Connections:
- no-connect marks 89 -> 0
Other:
- note removed: "**DCMI Alternate Function mappings** PA4 - HSYNC PB7 - VSYNC PA6 - PCLK PA9, PC6 - D0 PA10, PC7 - D1 PC8, PE0 - D2 PC9, PE1 - D3 PC11, PE4 - D4 PB6 - D5 PB8, PE5 - D6 PB9, PE6 - D7 PC10 - D8 PC12 - D9 PB5 - D10 PD2 - D11 PF11 - D12 PG15 - D13 **Available SPI AF Mappings** _SPI1_ (PA6 in use by OV) PA4, PA15 - NSS PA5, PB3 - SCK PB4 - MISO PA7, PB5 - MOSI _SPI2_ (MicroSD) PB12, PB9 - NSS PC3, PB15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"
- note removed: "Actual Product: 1987-DT024ETFT-IPS-SHB-ND 3-Line 9-bit Serial Comms IM[1:0] = 01; IM1(PA9) = LOW, IM0(PA8) = HIGH Using SPI3, RESET bound to PA2 GPIO"
- note removed: "CD - GPIO PB0"
- note removed: "RST - PE7 PWDWN - PE8"
- note removed: "SWCLK"
- note removed: "SWDIO"
- note removed: "TODO: 1. Add power supply 2. Assign XCLK 3. Calculate RGB LED Resistor values"
- title: STMCAM -> (none)

Commit message: restarted power
Other:
- added sheet Peripherals (pers.kicad_sch)
- added sheet Power_Conns (power_conns.kicad_sch)
- note added: "**DCMI Alternate Function mappings** PA4 - HSYNC PB7 - VSYNC PA6 - PCLK PA9, PC6 - D0 PA10, PC7 - D1 PC8, PE0 - D2 PC9, PE1 - D3 PC11, PE4 - D4 PB6 - D5 PB8, PE5 - D6 PB9, PE6 - D7 PC10 - D8 PC12 - D9 PB5 - D10 PD2 - D11 PF11 - D12 PG15 - D13 **Available SPI AF Mappings** _SPI1_ (PA6 in use by OV) PA4, PA15 - NSS PA5, PB3 - SCK PB4 - MISO PA7, PB5 - MOSI _SPI2_ (MicroSD) PB12, PB9 - NSS PC3, PB15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"
- note added: "TODO: 1. Add power supply 2. Assign XCLK 3. Reassign RGB LED Resistor values"
Changed lines of the file:
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@@
 	(generator "eeschema")
 	(generator_version "10.0")
-	(paper "A4")
+	(paper "A2")
+	(text "**DCMI Alternate Function mappings**\n\nPA4 - HSYNC \nPB7 - VSYNC \nPA6 - PCLK \nPA9, PC6 - D0 \nPA10, PC7 - D1\nPC8, PE0 - D2\nPC9, PE1 - D3\nPC11, PE4 - D4\nPB6 - D5 \nPB8, PE5 - D6\nPB9, PE6 - D7\nPC10 - D8 \nPC12 - D9\nPB5 - D10\nPD2 - D11\nPF11 - D12\nPG15 - D13\n\n\n**Available SPI AF Mappings**\n\n_SPI1_ (PA6 in use by OV)\nPA4, PA15 - NSS\nPA5, PB3 - SCK\nPB4 - MISO\nPA7, PB5 - MOSI\n\n_SPI2_ (MicroSD)\nPB12, PB9 - NSS\nPC3, PB15 - MOSI\nPB10, PB13 - SCK\nPB14, PC2 - MISO\n\n\n_SPI3_ (ILI9341)\nPA3, A15 - NSS\nPC10, PB3 - SCK\nPC11, PB4 - MISO\nPC12, PB5 - MOSI\n\n\n**I2C Mappings**\n\n_I2C 1_\nPB5 - SMBA\nPB6, PB8 - SCL\nPB7, PB9 - SDA\n\n\n_I2C 2_ (OV7670)\nPF0, PB11 - SDA\nPF1, PB10 - SCL\nPF2, PB12 - SMBA\n\n_I2C 3_ \nPC9 - SDA\nPA8 - SCL\nPA9 - SMBA\n\n\n\n\n\n"
+		(exclude_from_sim no)
+		(at 23.368 207.518 0)
+		(effects
+			(font
+				(size 1.905 1.905)
+			)
+			(justify left)
+		)
+	)
+	(text "TODO:\n1. Add power supply\n2. Assign XCLK\n3. Reassign RGB LED Resistor values\n"
+		(exclude_from_sim no)
+		(at 23.876 40.386 0)
+		(effects
+			(font
+				(size 5.08 5.08)
+			)
+			(justify left)
+		)
+	)
+	(sheet
+		(at 88.265 77.47)
+		(size 220.98 236.855)
+		(exclude_from_sim no)
+		(in_bom yes)
+		(on_board yes)
+		(dnp no)
+		(fields_autoplaced yes)
+		(stroke
+			(width 0.1524)
+			(type solid)
+		)
+		(fill
+			(color 0 0 0 0)
+		)
+		(property "Sheetname" "Peripherals"
+			(at 88.265 76.7584 0)
+			(show_name no)
+			(do_not_autoplace no)
+			(effects
+				(font
+					(size 1.27 1.27)
+				)
+				(justify left bottom)
+			)
+		)
+		(property "Sheetfile" "pers.kicad_sch"
+			(at 88.265 314.9096 0)
+			(show_name no)
+			(do_not_autoplace no)
+			(effects
+				(font
+					(size 1.27 1.27)
+				)
+				(justify left top)
+			)
+		)
+		(instances
+			(project "camCAD"
+				(path "/e2824ea6-9024-4cee-b80c-5fefbc7112d7"
+					(page "3")
+				)
+			)
+		)
+	)
+	(sheet
+		(at 337.82 76.835)
+		(size 215.265 142.24)
+		(exclude_from_sim no)
+		(in_bom yes)
+		(on_board yes)
+		(dnp no)
+		(fields_autoplaced yes)
+		(stroke
+			(width 0.1524)
+			(type solid)
+		)
+		(fill
+			(color 0 0 0 0)
+		)
+		(property "Sheetname" "Power_Conns"
+			(at 337.82 76.1234 0)
+			(show_name no)
+			(do_not_autoplace no)
+			(effects
+				(font
+					(size 1.27 1.27)
+				)
+				(justify left bottom)
+			)
+		)
+		(property "Sheetfile" "power_conns.kicad_sch"
+			(at 337.82 219.6596 0)
+			(show_name no)
+			(do_not_autoplace no)
+			(effects
+				(font
+					(size 1.27 1.27)
+				)
+				(justify left top)
+			)
+		)
+		(instances
+			(project "camCAD"
+				(path "/e2824ea6-9024-4cee-b80c-5fefbc7112d7"
+					(page "2")
+				)
+			)
+		)
+	)
 	(sheet_instances
 		(path "/"

Commit message: Included buck converter schematic
Other:
- sheet Peripherals renamed Chip_and_Peripherals
- sheet Power_Conns renamed Power_Supply_Scheme
- added sheet Buck_Converter (buck.kicad_sch)
Changed lines of the file:
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@@
 			(color 0 0 0 0)
 		)
-		(property "Sheetname" "Peripherals"
+		(property "Sheetname" "Chip_and_Peripherals"
 			(at 88.265 76.7584 0)
 			(show_name no)
@@
 	)
 	(sheet
+		(at 338.455 236.855)
+		(size 213.995 77.47)
+		(exclude_from_sim no)
+		(in_bom yes)
+		(on_board yes)
+		(dnp no)
+		(fields_autoplaced yes)
+		(stroke
+			(width 0.1524)
+			(type solid)
+		)
+		(fill
+			(color 0 0 0 0)
+		)
+		(property "Sheetname" "Buck_Converter"
+			(at 338.455 236.1434 0)
+			(show_name no)
+			(do_not_autoplace no)
+			(effects
+				(font
+					(size 1.27 1.27)
+				)
+				(justify left bottom)
+			)
+		)
+		(property "Sheetfile" "buck.kicad_sch"
+			(at 338.455 314.9096 0)
+			(show_name no)
+			(do_not_autoplace no)
+			(effects
+				(font
+					(size 1.27 1.27)
+				)
+				(justify left top)
+			)
+		)
+		(instances
+			(project "camCAD"
+				(path "/e2824ea6-9024-4cee-b80c-5fefbc7112d7"
+					(page "4")
+				)
+			)
+		)
+	)
+	(sheet
 		(at 337.82 76.835)
 		(size 215.265 142.24)
@@
 			(color 0 0 0 0)
 		)
-		(property "Sheetname" "Power_Conns"
+		(property "Sheetname" "Power_Supply_Scheme"
 			(at 337.82 76.1234 0)
 			(show_name no)
