File: camCAD/camCAD.kicad_sch (KiCad schematic)
At the start: 0 parts

Commit message: Push post-print
Other:
- note removed: "TODO: 1. REWIRE a. SPI for display needs to use PA15 b. Add a 18-pin header for EYESPI connector instead"
Changed lines of the file:
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@@
 		(comment 4 "By Siddharth Vasudevan")
 	)
-	(text "TODO:\n1. REWIRE\n	a. SPI for display needs to use PA15\n	b. Add a 18-pin header for EYESPI connector instead\n	"
+	(text ""
 		(exclude_from_sim no)
 		(at 192.278 173.99 0)
