File: camCAD/_autosave-buck.kicad_sch (KiCad schematic)
At the start: 19 parts, among them J1 USB C Charging Port, J3 BATTERY, U1 BQ24072RGTR Charging IC, U2 SC189ZSKTRT

Commit message: Started PCB Layout, need to add a user interface
Connections:
- net BQ_CHG: now also D7.C (K); no longer D7.1 (K)
- net BQ_PGOOD: now also D6.C (K); no longer D6.1 (K)
- net at R10.2: now also D6.A; no longer D6.2 (A)
- net at R12.2: now also D7.A; no longer D7.2 (A)
Changed lines of the file:
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@@
 			)
 		)
-		(pin "1"
-		)
-		(pin "2"
+		(pin "C"
+		)
+		(pin "A"
 		)
 		(instances
@@
 	)
 	(symbol
+		(lib_name "LED_1")
 		(lib_id "Device:LED")
 		(at 97.79 109.22 90)
@@
 			)
 		)
-		(pin "1"
-		)
-		(pin "2"
-		)
-		(instances
+		(pin "C"
+		)
+		(pin "A"
+		)
+		(instances
