File: camCAD/components.kicad_sch (KiCad schematic)
At the start: 13 parts, among them J4 ILI9341_Display_Header, SW2 SW_Push

Commit message: Nearly done with DPPM connections, updated readme
Parts:
- removed D1: LED1, symbol Device:LED
- removed D2: LED2, symbol Device:LED
- removed R3, R4: 6.8K, symbol Device:R_Small_US
- D3: value Activity+PowerLED -> ActivityLED
Other:
- moved on the sheet: R1, SW2, Z1

Commit message: miscellaneous changes
Parts:
- removed R1: R_US, symbol Device:R_US
- removed SW2: SW_Push, symbol Switch:SW_Push
- added C27: 1uF, symbol Device:C
- added C28, C29: 1uF cer, low ESR, symbol Device:C
- added U4: AP3602AKTR-G1 Charge Pump, SOT-23-6_DIO, symbol 1_ChargePump:AP3602AKTR-G1
- added U5: (no value), symbol 1_LEDs:QBLP677AD-IWD-2897
- R5: value TBD -> 22
- R6: value TBD -> 33
- R7: value TBD -> 56
Connections:
- net GND: now also C28.2, C29.2, U4.2 (GND), U5.1, U5.3, U5.4
- net PB11: now reaches OV2.P$13 (XCLK)
- net +3.3V renamed AP_VIN
- net AP_VIN: now also C29.1, U4.3 (*SHDN), U4.5 (VIN)
- net PB3 renamed PA5
- new net: C27.2, U4.4 (C-)
- new net: C27.1, U4.6 (C+)
- new net AP_VOUT: C28.1, U4.1 (VOUT), U5.2 (A)
Other:
- note added: "AP3602A Charge Pump + Flash LED"
- note added: "Product: 1987-DT024ETFT-IPS-SHB-ND 3-Line 9-bit Serial Comms IM[1:0] = 01; IM1(PA9) = LOW, IM0(PA8) = HIGH {This should be set in software} Using SPI3, RESET bound to PA2 GPIO"
- note removed: "Actual Product: 1987-DT024ETFT-IPS-SHB-ND 3-Line 9-bit Serial Comms IM[1:0] = 01; IM1(PA9) = LOW, IM0(PA8) = HIGH {This should be set in software} Using SPI3, RESET bound to PA2 GPIO"
- note removed: "Bootloader mode switch"
- moved on the sheet: D3, R5, R6, R7, Z1

Commit message: Added footprints for major components, renamed some components for more specific information
Parts:
- removed Z1: MicroSD_Breakout, symbol 1_MicroSD:MicroSD_BREA
- added U6: ADA 254, 1_MicroSD:MODULE_254, symbol 1_MicroSD:254
- C27: value 1uF -> 1uF cer, low ESR
- D3: footprint CLMVC-FKA-CL1D1L71BB7C3C3_CRE -> 1_LEDs:CLMVC-FKA-CL1D1L71BB7C3C3_CRE
- J4: footprint 5051101592:CON_5051101592_MOL -> 1_Headers:CON_5051101592_MOL
- OV2: footprint CAMERA-OV7670:CAMERA-OV7670-DIP -> 1_Cameras:CAMERA-OV7670-DIP
- U4: footprint SOT-23-6_DIO -> 1_ChargePump:SOT-23-6_DIO
- U5: value (none) -> Flash LED; footprint (none) -> 1_LEDs:QBLP677AD-IWD-2897
Connections:
- net AP_VIN: now also U6.7 (3V)
- net GND: now also U6.6 (GND)
- net PB0: now also U6.1 (CD)
- net PB12: now also U6.2 (CS)
- net PB13: now also U6.5 (CLK)
- net PB14: now also U6.4 (DO)
- net PB15: now also U6.3 (DI)
- no-connect marks 4 -> 5
Other:
- note added: "Adafruit MicroSD Breakout Board"
- note removed: "MicroSD Transflash Breakout Board"

Commit message: Started PCB Layout, need to add a user interface
Parts:
- C27, C28, C29: footprint (none) -> Capacitor_SMD:C_0603_1608Metric
- R5, R6, R7: footprint (none) -> Resistor_SMD:R_0402_1005Metric
Changed lines of the file:
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@@
 			)
 		)
-		(property "Footprint" ""
+		(property "Footprint" "Capacitor_SMD:C_0603_1608Metric"
 			(at 233.3752 76.2 0)
 			(hide yes)
@@
 			)
 		)
-		(property "Footprint" ""
+		(property "Footprint" "Resistor_SMD:R_0402_1005Metric"
 			(at 43.18 110.49 0)
 			(hide yes)
@@
 			)
 		)
-		(property "Footprint" ""
+		(property "Footprint" "Capacitor_SMD:C_0603_1608Metric"
 			(at 243.5352 40.64 0)
 			(hide yes)
@@
 			)
 		)
-		(property "Footprint" ""
+		(property "Footprint" "Resistor_SMD:R_0402_1005Metric"
 			(at 43.18 105.41 0)
 			(hide yes)
@@
 			)
 		)
-		(property "Footprint" ""
+		(property "Footprint" "Capacitor_SMD:C_0603_1608Metric"
 			(at 201.6252 83.82 0)
 			(hide yes)
@@
 			)
 		)
-		(property "Footprint" ""
+		(property "Footprint" "Resistor_SMD:R_0402_1005Metric"
 			(at 43.18 107.95 0)
 			(hide yes)
