File: camCAD/power_conns.kicad_sch (KiCad schematic)
At the start: 22 parts, among them SW1 SW_Push

Commit message: Nearly done with DPPM connections, updated readme
Parts:
- renumbered 100K to 100K1
Connections:
- net BUCK3.3V renamed BUCKOUT
Changed lines of the file:
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@@
 		)
 	)
-	(global_label "BUCK3.3V"
+	(global_label "BUCKOUT"
 		(shape input)
 		(at 97.79 20.32 0)
@@
 		)
 		(property "Intersheetrefs" "${INTERSHEET_REFS}"
-			(at 110.0281 20.32 0)
-			(hide yes)
-			(show_name no)
-			(do_not_autoplace no)
-			(effects
-				(font
-					(size 1.27 1.27)
-				)
-				(justify left)
-			)
-		)
-	)
-	(global_label "BUCK3.3V"
+			(at 109.5443 20.32 0)
+			(hide yes)
+			(show_name no)
+			(do_not_autoplace no)
+			(effects
+				(font
+					(size 1.27 1.27)
+				)
+				(justify left)
+			)
+		)
+	)
+	(global_label "BUCKOUT"
 		(shape input)
 		(at 39.37 96.52 0)
@@
 		)
 		(property "Intersheetrefs" "${INTERSHEET_REFS}"
-			(at 51.6081 96.52 0)
+			(at 51.1243 96.52 0)
 			(hide yes)
 			(show_name no)
@@
 		)
 	)
-	(global_label "BUCK3.3V"
+	(global_label "BUCKOUT"
 		(shape input)
 		(at 93.98 106.68 180)
@@
 		)
 		(property "Intersheetrefs" "${INTERSHEET_REFS}"
-			(at 81.7419 106.68 0)
+			(at 82.2257 106.68 0)
 			(hide yes)
 			(show_name no)
@@
 		(in_pos_files yes)
 		(dnp no)
-		(property "Reference" "100K"
+		(property "Reference" "100K1"
 			(at 102.489 102.743 90)
 			(show_name no)
@@
 			(project "camCAD"
 				(path "/e2824ea6-9024-4cee-b80c-5fefbc7112d7/da932f2b-e136-46c9-98f4-43086828212d"
-					(reference "100K")
+					(reference "100K1")
 					(unit 1)
 				)

Commit message: miscellaneous changes
Parts:
- removed 100K1: R_Small_US, symbol Device:R_Small_US
- removed FB1: 600 Ohm @ 100MHz, symbol Device:FerriteBead
- added C22: 1uF, symbol Device:C
- added C23: 100nF, symbol Device:C
- added FB1: FerriteBead_Small, symbol Device:FerriteBead_Small
- added R8: 47, symbol Device:R_Small_US
- C19: value 100nF -> 0.1uF
Connections:
- net GND: now also C3.2, SW1.1, C23.2; no longer C10.2, C11.2, C12.2, C13.2, C14.2, C15.2, C4.2, C5.2, C6.2, C7.2, C8.2, C9.2
- net NRST: now also C19.1
- net BUCKOUT renamed SC_3V3
- net SC_3V3: now also C10.1, FB1.1, R8.2; no longer C3.1
- removed net VDD7: C10.1, C3.2
- net VDDA: no longer names the net of C16.1
- net VDDA: now also FB1.2
- new net: C10.2, C11.2, C12.2, C13.2, C14.2, C15.2, C3.1, C4.2, C5.2, C6.2, C7.2, C8.2, C9.2
- new net: C22.2, C23.1
- new net VREF+: C22.1, R8.1
Other:
- note added: "NRST protection circuit"
- note added: "VCAPx and VREF+ connections"
- note removed: "NRST connection"
- note removed: "VCAPx connections"
- moved on the sheet: C1, C10, C11, C12, C13, C14, C15, C16, C17, C18, C19, C2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

Commit message: Added footprints for major components, renamed some components for more specific information
Parts:
- C1, C2: value 2.2uF -> 2.2uF cer
- C10, C11, C12, C13, C14, C15, C17, C18, C23, C4, C5, C6, C7, C8, C9: value 100nF -> 100nF cer
- C16, C22: value 1uF -> 1uF cer
- C3: value 4.7uF -> 4.7uF cer
- FB1: footprint (none) -> 1_FerriteBeads:BEADC1608X95N
- SW1: footprint (none) -> 1_Switches:SW_SKRPABE010
Changed lines of the file:
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@@
 			)
 		)
-		(property "Value" "100nF"
+		(property "Value" "100nF cer"
 			(at 88.9 46.9899 0)
 			(show_name no)
@@
 			)
 		)
-		(property "Value" "100nF"
+		(property "Value" "100nF cer"
 			(at 171.45 46.9899 0)
 			(show_name no)
@@
 			)
 		)
-		(property "Value" "4.7uF"
+		(property "Value" "4.7uF cer"
 			(at 101.6 64.7699 0)
 			(show_name no)
@@
 			)
 		)
-		(property "Value" "100nF"
+		(property "Value" "100nF cer"
 			(at 58.42 129.5399 0)
 			(show_name no)
@@
 			)
 		)
-		(property "Value" "100nF"
+		(property "Value" "100nF cer"
 			(at 62.23 46.9899 0)
 			(show_name no)
@@
 			)
 		)
-		(property "Value" "100nF"
+		(property "Value" "100nF cer"
 			(at 22.86 46.9899 0)
 			(show_name no)
@@
 			)
 		)
-		(property "Value" "100nF"
+		(property "Value" "100nF cer"
 			(at 185.42 118.1099 0)
 			(show_name no)
@@
 			)
 		)
-		(property "Value" "100nF"
+		(property "Value" "100nF cer"
 			(at 143.51 46.9899 0)
 			(show_name no)
@@
 			)
 		)
-		(property "Value" "100nF"
+		(property "Value" "100nF cer"
 			(at 26.67 142.2399 0)
 			(show_name no)
@@
 			)
 		)
-		(property "Value" "2.2uF"
+		(property "Value" "2.2uF cer"
 			(at 144.78 118.1099 0)
 			(show_name no)
@@
 			)
 		)
-		(property "Value" "100nF"
+		(property "Value" "100nF cer"
 			(at 74.93 46.9899 0)
 			(show_name no)
@@
 			)
 		)
-		(property "Value" "1uF"
+		(property "Value" "1uF cer"
 			(at 185.42 109.2199 0)
 			(show_name no)
@@
 			)
 		)
-		(property "Footprint" ""
+		(property "Footprint" "1_Switches:SW_SKRPABE010"
 			(at 82.55 114.3 0)
 			(hide yes)
@@
 			)
 		)
-		(property "Value" "100nF"
+		(property "Value" "100nF cer"
 			(at 49.53 46.9899 0)
 			(show_name no)
@@
 			)
 		)
-		(property "Value" "100nF"
+		(property "Value" "100nF cer"
 			(at 157.48 46.9899 0)
 			(show_name no)
@@
 			)
 		)
-		(property "Value" "1uF"
+		(property "Value" "1uF cer"
 			(at 26.67 133.3499 0)
 			(show_name no)
@@
 			)
 		)
-		(property "Value" "2.2uF"
+		(property "Value" "2.2uF cer"
 			(at 158.75 118.1099 0)
 			(show_name no)
@@
 			)
 		)
-		(property "Value" "100nF"
+		(property "Value" "100nF cer"
 			(at 35.56 46.9899 0)
 			(show_name no)
@@
 			)
 		)
-		(property "Value" "100nF"
+		(property "Value" "100nF cer"
 			(at 129.54 46.9899 0)
 			(show_name no)
@@
 			)
 		)
-		(property "Value" "100nF"
+		(property "Value" "100nF cer"
 			(at 101.6 46.9899 0)
 			(show_name no)
@@
 			)
 		)
-		(property "Footprint" ""
+		(property "Footprint" "1_FerriteBeads:BEADC1608X95N"
 			(at 21.082 120.65 90)
 			(hide yes)
@@
 			)
 		)
-		(property "Value" "100nF"
+		(property "Value" "100nF cer"
 			(at 115.57 46.9899 0)
 			(show_name no)

Commit message: Started PCB Layout, need to add a user interface
Parts:
- C1, C2: footprint (none) -> Capacitor_SMD:C_0201_0603Metric
- C10, C11, C12, C13, C14, C15, C16, C17, C18, C19, C22, C23, C4, C5, C6, C7, C8, C9: footprint (none) -> Capacitor_SMD:C_0603_1608Metric
- C3: footprint (none) -> Capacitor_SMD:C_0805_2012Metric
- R8: footprint (none) -> Resistor_SMD:R_1206_3216Metric
Changed lines of the file:
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@@
 			)
 		)
-		(property "Footprint" ""
+		(property "Footprint" "Capacitor_SMD:C_0603_1608Metric"
 			(at 86.0552 49.53 0)
 			(hide yes)
@@
 			)
 		)
-		(property "Footprint" ""
+		(property "Footprint" "Resistor_SMD:R_1206_3216Metric"
 			(at 186.69 104.14 0)
 			(hide yes)
@@
 			)
 		)
-		(property "Footprint" ""
+		(property "Footprint" "Capacitor_SMD:C_0603_1608Metric"
 			(at 168.6052 49.53 0)
 			(hide yes)
@@
 			)
 		)
-		(property "Footprint" ""
+		(property "Footprint" "Capacitor_SMD:C_0805_2012Metric"
 			(at 98.7552 67.31 0)
 			(hide yes)
@@
 			)
 		)
-		(property "Footprint" ""
+		(property "Footprint" "Capacitor_SMD:C_0603_1608Metric"
 			(at 102.5652 119.38 0)
 			(hide yes)
@@
 			)
 		)
-		(property "Footprint" ""
+		(property "Footprint" "Capacitor_SMD:C_0603_1608Metric"
 			(at 55.5752 132.08 0)
 			(hide yes)
@@
 			)
 		)
-		(property "Footprint" ""
+		(property "Footprint" "Capacitor_SMD:C_0603_1608Metric"
 			(at 59.3852 49.53 0)
 			(hide yes)
@@
 			)
 		)
-		(property "Footprint" ""
+		(property "Footprint" "Capacitor_SMD:C_0603_1608Metric"
 			(at 20.0152 49.53 0)
 			(hide yes)
@@
 			)
 		)
-		(property "Footprint" ""
+		(property "Footprint" "Capacitor_SMD:C_0603_1608Metric"
 			(at 182.5752 120.65 0)
 			(hide yes)
@@
 			)
 		)
-		(property "Footprint" ""
+		(property "Footprint" "Capacitor_SMD:C_0603_1608Metric"
 			(at 140.6652 49.53 0)
 			(hide yes)
@@
 			)
 		)
-		(property "Footprint" ""
+		(property "Footprint" "Capacitor_SMD:C_0603_1608Metric"
 			(at 23.8252 144.78 0)
 			(hide yes)
@@
 			)
 		)
-		(property "Footprint" ""
+		(property "Footprint" "Capacitor_SMD:C_0201_0603Metric"
 			(at 141.9352 120.65 0)
 			(hide yes)
@@
 			)
 		)
-		(property "Footprint" ""
+		(property "Footprint" "Capacitor_SMD:C_0603_1608Metric"
 			(at 72.0852 49.53 0)
 			(hide yes)
@@
 			)
 		)
-		(property "Footprint" ""
+		(property "Footprint" "Capacitor_SMD:C_0603_1608Metric"
 			(at 182.5752 111.76 0)
 			(hide yes)
@@
 			)
 		)
-		(property "Footprint" ""
+		(property "Footprint" "Capacitor_SMD:C_0603_1608Metric"
 			(at 46.6852 49.53 0)
 			(hide yes)
@@
 			)
 		)
-		(property "Footprint" ""
+		(property "Footprint" "Capacitor_SMD:C_0603_1608Metric"
 			(at 154.6352 49.53 0)
 			(hide yes)
@@
 			)
 		)
-		(property "Footprint" ""
+		(property "Footprint" "Capacitor_SMD:C_0603_1608Metric"
 			(at 23.8252 135.89 0)
 			(hide yes)
@@
 			)
 		)
-		(property "Footprint" ""
+		(property "Footprint" "Capacitor_SMD:C_0201_0603Metric"
 			(at 157.1752 120.65 0)
 			(hide yes)
@@
 			)
 		)
-		(property "Footprint" ""
+		(property "Footprint" "Capacitor_SMD:C_0603_1608Metric"
 			(at 32.7152 49.53 0)
 			(hide yes)
@@
 			)
 		)
-		(property "Footprint" ""
+		(property "Footprint" "Capacitor_SMD:C_0603_1608Metric"
 			(at 126.6952 49.53 0)
 			(hide yes)
@@
 			)
 		)
-		(property "Footprint" ""
+		(property "Footprint" "Capacitor_SMD:C_0603_1608Metric"
 			(at 98.7552 49.53 0)
 			(hide yes)
@@
 			)
 		)
-		(property "Footprint" ""
+		(property "Footprint" "Capacitor_SMD:C_0603_1608Metric"
 			(at 112.7252 49.53 0)
 			(hide yes)

Commit message: Rearranged layout
Parts:
- SW1: value SW_Push -> NRST_SW
Changed lines of the file:
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@@
 			)
 		)
-		(property "Value" "SW_Push"
+		(property "Value" "NRST_SW"
 			(at 88.9 115.5699 90)
 			(show_name no)
