File: camCAD/power_conns.kicad_sch (KiCad schematic)
At the start: 24 parts, among them SW1 NRST_SW

Commit message: Random push ishan karne
Connections:
- net C10-: now reaches C10.2, C11.2, C12.2, C13.2, C14.2, C15.2, C3.1, C4.2, C5.2, C6.2, C7.2, C8.2, C9.2
Changed lines of the file:
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@@
+	(wire
+		(pts
+			(xy 97.79 55.88) (xy 111.76 55.88)
+		)
+		(stroke
+			(width 0)
+			(type default)
+		)
+	)
 	(wire
 		(pts
@@
 	(wire
 		(pts
-			(xy 97.79 55.88) (xy 111.76 55.88)
-		)
-		(stroke
-			(width 0)
-			(type default)
-		)
-	)
-	(wire
-		(pts
 			(xy 22.86 144.78) (xy 22.86 153.67)
 		)
@@
 		)
 	)
+	(label "C10-"
+		(at 97.79 55.88 0)
+		(effects
+			(font
+				(size 1.27 1.27)
+			)
+			(justify left bottom)
+		)
+	)

Commit message: layout partially complete
Connections:
- net C10- renamed CapJunction
Changed lines of the file:
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@@
 		)
 	)
-	(label "C10-"
+	(label "CapJunction"
 		(at 97.79 55.88 0)
 		(effects
