File: camCAD/_autosave-components.kicad_sch (KiCad schematic)
At the start: 12 parts, among them J4 ILI9341_Display_Header, U4 AP3602AKTR-G1 Charge Pump, U5 Flash LED, U6 ADA 254

Commit message: Random push ishan karne
Changed lines of the file:
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@@
 	(wire
 		(pts
-			(xy 27.94 57.15) (xy 34.29 57.15)
+			(xy 30.48 57.15) (xy 34.29 57.15)
 		)
 		(stroke
@@
 	(global_label "SC_3V3"
 		(shape input)
-		(at 27.94 57.15 180)
+		(at 30.48 57.15 180)
 		(fields_autoplaced yes)
 		(effects
@@
 		)
 		(property "Intersheetrefs" "${INTERSHEET_REFS}"
-			(at 18.0001 57.15 0)
+			(at 20.5401 57.15 0)
 			(hide yes)
 			(show_name no)
