File: camCAD/camCAD.kicad_pcb (KiCad board)
At the start: 2 copper layers, 58 parts, among them J1 USB C Charging Port, J2 JTAG header, J3 BATTERY, J4 ILI9341_Display_Header, SW1 SW_Push, U1 BQ24072RGTR Charging IC, U2 SC189ZSKTRT, U3 STM32F407ZGTx, U4 AP3602AKTR-G1 Charge Pump, U5 Flash LED, U6 ADA 254

Commit message: Rearranged layout
Parts:
- added R14: 10k, Resistor_SMD:R_0402_1005Metric, F.Cu at (62.0, 47.1)
- added R15: 10k, Resistor_SMD:R_0402_1005Metric, F.Cu at (62.0, 49.1)
- added R16: 10k, Resistor_SMD:R_0402_1005Metric, F.Cu at (62.0, 51.1)
- added R17: 10k, Resistor_SMD:R_0402_1005Metric, F.Cu at (62.0, 53.1)
- added R18: 100k, Resistor_SMD:R_0402_1005Metric, F.Cu at (149.3, 51.1)
- added R19: 220k, Resistor_SMD:R_0805_2012Metric, F.Cu at (146.5, 51.0)
- added R9: 10k, Resistor_SMD:R_0402_1005Metric, F.Cu at (62.0, 45.1)
- added SW2: Pictures/Back, 1_Switches:SW_SKRPABE010, F.Cu at (57.1, 46.5)
- added SW3: Forward, 1_Switches:SW_SKRPABE010, F.Cu at (57.1, 51.2)
- added SW4: Backward, 1_Switches:SW_SKRPABE010, F.Cu at (57.1, 56.0)
- added SW5: Flash/Delete, 1_Switches:SW_SKRPABE010, F.Cu at (57.1, 60.7)
- added SW6: Shutter, 1_Switches:SW_SKRPABE010, F.Cu at (57.1, 65.5)
- SW1: value SW_Push -> NRST_SW
- moved U6 118.6 mm to (100.5, 99.1), turned to 90 degrees
- moved C1 112.0 mm to (86.1, 45.2)
- moved C2 112.0 mm to (85.3, 47.2)
- moved C3 111.7 mm to (88.8, 58.6), turned to 90 degrees
- moved D3 101.0 mm to (74.7, 58.3), turned to 90 degrees
- moved R8 100.6 mm to (129.8, 48.2)
- moved C20 98.0 mm to (123.8, 54.5), turned to 0 degrees
- moved C18 93.6 mm to (127.0, 54.5)
- moved R5 92.3 mm to (79.5, 54.5), turned to 180 degrees
- moved C21 92.2 mm to (123.8, 52.2)
- moved R6 91.5 mm to (79.5, 58.1), turned to 180 degrees
- moved L1 91.3 mm to (130.7, 51.7)
- moved R7 91.2 mm to (79.5, 61.7), turned to 180 degrees
- moved U2 89.9 mm to (126.9, 51.5)
- moved C23 88.8 mm to (118.5, 53.9)
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Connections:
- U3 pad 13: unconnected-(U3-PF3-Pad13) -> PF3
- U3 pad 57: unconnected-(U3-PG1-Pad57) -> PG1
- U3 pad 87: unconnected-(U3-PG2-Pad87) -> PG2
- U3 pad 88: unconnected-(U3-PG3-Pad88) -> PG3
- U3 pad 89: unconnected-(U3-PG4-Pad89) -> PG4
- U3 pad 90: unconnected-(U3-PG5-Pad90) -> PG5
Routing:
- net AP_VIN: track 0.00 -> 14.8 mm
- net BATT-: track 0.00 -> 12.8 mm
- net BQ_OUT: track 0.00 -> 7.78 mm
- net Net-(J1-CC1): track 0.00 -> 1.74 mm

Commit message: Random push ishan karne
Parts:
- D3, D6, D7, J1, J2, J3, J4, SW1, SW2, SW3, SW4, SW5, U6: moved to B.Cu
- moved SW2 71.3 mm to (90.4, 109.5), turned to 180 degrees
- moved SW3 67.4 mm to (97.5, 105.2), turned to 180 degrees
- moved U6 63.4 mm to (156.9, 70.0), turned to 180 degrees
- moved SW5 63.3 mm to (97.5, 109.5), turned to 180 degrees
- moved SW4 59.4 mm to (90.3, 105.2), turned to 180 degrees
- moved J2 56.2 mm to (97.6, 96.8), turned to 180 degrees
- moved SW1 51.1 mm to (90.3, 89.3), turned to 0 degrees
- moved J1 46.2 mm to (168.1, 111.0), turned to 180 degrees
- moved C21 45.3 mm to (165.4, 70.2), turned to 180 degrees
- moved U2 44.8 mm to (166.2, 73.1)
- moved L1 44.8 mm to (170.0, 73.2)
- moved R9 44.5 mm to (103.4, 61.5), turned to 90 degrees
- moved C20 43.9 mm to (163.2, 73.8), turned to 90 degrees
- moved R18 40.3 mm to (118.2, 76.7)
- moved R19 39.0 mm to (118.6, 78.3), turned to 0 degrees
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Connections:
- net AP_VIN renamed SC_3V3
- net Net-(C10-Pad2) renamed /STM32_Power_Requirements/C10-
- U1 pad V: (no net) -> BATT-
Routing:
- net /STM32_Power_Requirements/C10-: track 0.00 -> 14.4 mm
- net SC_3V3: track 14.8 -> 22.9 mm
- net BQ_OUT: track 7.78 -> 0.00 mm
- net PF3: track 0.00 -> 4.31 mm
- net VREF+: track 0.00 -> 2.22 mm
- net BATT-: track 12.8 -> 10.6 mm
- net BOOT0: track 0.00 -> 1.85 mm
- net Net-(J1-CC1): track 1.74 -> 0.00 mm
Other:
- board text added: "."

Commit message: layout partially complete
Parts:
- C27, C28, C29, OV2, SW6, U4, U5: moved to B.Cu
- D3, D6, D7, J1, J2, J3, J4, SW1, SW2, SW3, SW4, SW5, U6: moved to F.Cu
- moved J3 91.0 mm to (73.8, 58.0)
- moved C26 89.2 mm to (88.7, 51.6), turned to 90 degrees
- moved R13 88.3 mm to (87.1, 51.9), turned to 90 degrees
- moved C24 88.2 mm to (83.3, 55.8), turned to 180 degrees
- moved U1 87.9 mm to (87.9, 55.7)
- moved R11 87.3 mm to (91.3, 55.0), turned to 0 degrees
- moved R4 86.8 mm to (85.7, 52.0), turned to -90 degrees
- moved R12 86.0 mm to (87.2, 93.9)
- moved R10 84.6 mm to (87.2, 97.2)
- moved C25 83.9 mm to (87.6, 60.1), turned to -90 degrees
- moved D7 74.3 mm to (88.9, 93.8)
- moved D6 74.2 mm to (88.9, 97.2)
- moved R2 73.1 mm to (98.3, 89.4), turned to 180 degrees
- moved SW6 69.9 mm to (158.2, 52.9), turned to 0 degrees
- moved J1 68.1 mm to (101.0, 100.0), turned to 0 degrees
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Connections:
- net /STM32_Power_Requirements/C10- renamed /STM32_Power_Requirements/CapJunction
- U1 pad V: BATT- -> (no net)
Routing:
- net SC_3V3: track 22.9 -> 221.4 mm, vias 0 -> 3
- net BATT-: track 10.6 -> 178.1 mm, vias 0 -> 2
- net /STM32_Power_Requirements/CapJunction: track 14.4 -> 93.5 mm, vias 0 -> 9
- net PG5: track 0.00 -> 74.8 mm, vias 0 -> 1
- net BQ_OUT: track 0.00 -> 62.8 mm, vias 0 -> 2
- net NRST: track 0.00 -> 57.1 mm, vias 0 -> 2
- net PG4: track 0.00 -> 53.1 mm
- net BQ_IN: track 0.00 -> 53.1 mm, vias 0 -> 2
- net PG1: track 0.00 -> 52.9 mm, vias 0 -> 2
- net PA5: track 0.00 -> 51.4 mm, vias 0 -> 2
- net PA9: track 0.00 -> 51.2 mm, vias 0 -> 2
- net PG3: track 0.00 -> 50.2 mm
- net PA8: track 0.00 -> 50.2 mm, vias 0 -> 2
- net Net-(D3-R): track 0.00 -> 45.9 mm, vias 0 -> 2
- net PG2: track 0.00 -> 44.1 mm, vias 0 -> 2
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- added copper zone on B.Cu, net BATT-
- added copper zone on F.Cu, net BATT-
- added copper zone on F.Cu, net SC_3V3

Commit message: Modified pcb layout
Routing:
- net BATT+: track 13.7 -> 142.5 mm, vias 0 -> 2
- net BATT-: track 178.1 -> 228.8 mm, vias 2 -> 8
- net SC_3V3: track 221.4 -> 269.8 mm, vias 3 -> 7
- net PB7: track 36.1 -> 35.4 mm
- net /STM32_Power_Requirements/CapJunction: track 93.5 -> 93.6 mm, vias 9 -> 10
- removed copper zone on F.Cu, net BATT-
