File: camCAD/_autosave-camCAD_fourLayer.kicad_pcb (KiCad board)
At the start: 4 copper layers, 89 x 54.6 mm, 70 parts, among them J1 USB C Charging Port, J2 JTAG header, J3 BATTERY, J4 ILI9341_Display_Header, SW1 NRST_SW, SW2 Pictures/Back, SW3 Forward, SW4 Backward, SW5 Flash/Delete, SW6 Shutter, U1 BQ24072RGTR Charging IC, U2 SC189ZSKTRT, U3 STM32F407ZGTx, U4 AP3602AKTR-G1 Charge Pump, U5 Flash LED, U6 ADA 254

Commit message: Added some decor
Other:
- board text added: "熊猫"
