File: camCAD/camCAD_fourLayer_v2.kicad_pcb (KiCad board)
At the start: 4 copper layers, 87.6 x 54.6 mm, 70 parts, among them J1 USB C Charging Port, J2 SWD Header, J3 BATTERY, J4 EYESPI, SW1 NRST_SW, SW2 Pictures/Back, SW3 Forward, SW4 Backward, SW5 Flash/Delete, SW6 Shutter, U1 BQ24072RGTR Charging IC, U2 SC189ZSKTRT, U3 STM32F407ZGTx, U4 AP3602AKTR-G1 Charge Pump, U5 Flash LED, U6 ADA 254

Commit message: Push post-print
Parts:
- moved C16 52.5 mm to (100.1, 38.0)
- moved FB1 52.5 mm to (96.7, 38.1)
- moved C18 52.5 mm to (97.1, 54.6)
- moved D3 52.5 mm to (36.8, 65.3)
- moved R2 52.5 mm to (52.1, 64.4)
- moved C1 52.5 mm to (76.2, 36.1)
- moved C12 52.5 mm to (69.3, 53.4)
- moved C13 52.5 mm to (85.6, 61.6)
- moved C14 52.5 mm to (80.6, 61.6)
- moved C15 52.5 mm to (69.4, 57.0)
- moved C17 52.5 mm to (100.1, 35.2)
- moved C2 52.5 mm to (70.1, 55.4)
- moved C20 52.5 mm to (54.3, 31.3)
- moved C22 52.5 mm to (96.7, 41.0)
- moved C23 52.5 mm to (100.0, 41.0)
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Routing:
- net PE0: track 27.4 -> 25.2 mm, vias 2 -> 1
- net Net-(D3-R): track 42.1 -> 42.6 mm
- net PG1: track 59.6 -> 60.1 mm
- net NRST: vias 3 -> 2
